Commit message: Complete diffdrive, arm and rocker_bogie
Warehouse_simulation launch file can now run two robot simultaniously
Examined the correctness of DH table in script mim_arm.py

File: urdf/diffdrive/mim_diffdrive.urdf (robot description, URDF)
Before this commit: robot mim_diffdrive, 11 links, 10 joints
Links:
- added link LIDAR, mass 0.0730843683225071; collision mesh filename=package://mim_robots/meshes/diffdrive/LIDAR.STL; visual mesh filename=package://mim_robots/meshes/diffdrive/LIDAR.STL
- link C1: mass 0.0171596756026443 -> 0.133845469700625; geometry collision mesh filename=package://mim_robots/meshes/diffdrive/C1.STL; visual mesh filename=package://mim_robots/meshes/diffdrive/C1.STL
- link C1W: mass 0.0741004703095722 -> 0.0290199529351017; geometry collision mesh filename=package://mim_robots/meshes/diffdrive/C1W.STL; visual mesh filename=package://mim_robots/meshes/diffdrive/C1W.STL
- link C2: mass 0.0171596756026444 -> 0.133845469700627; geometry collision mesh filename=package://mim_robots/meshes/diffdrive/C2.STL; visual mesh filename=package://mim_robots/meshes/diffdrive/C2.STL
- link C2W: mass 0.0741004703095722 -> 0.0290199529351017; geometry collision mesh filename=package://mim_robots/meshes/diffdrive/C2W.STL; visual mesh filename=package://mim_robots/meshes/diffdrive/C2W.STL
- link C3: mass 0.0171596756026444 -> 0.133845469700626; geometry collision mesh filename=package://mim_robots/meshes/diffdrive/C3.STL; visual mesh filename=package://mim_robots/meshes/diffdrive/C3.STL
- link C3W: mass 0.0741004703095722 -> 0.0290199529351017; geometry collision mesh filename=package://mim_robots/meshes/diffdrive/C3W.STL; visual mesh filename=package://mim_robots/meshes/diffdrive/C3W.STL
- link C4: mass 0.0171596756026442 -> 0.133845469700625; geometry collision mesh filename=package://mim_robots/meshes/diffdrive/C4.STL; visual mesh filename=package://mim_robots/meshes/diffdrive/C4.STL
- link C4W: mass 0.0741004703095722 -> 0.0290199529351017; geometry collision mesh filename=package://mim_robots/meshes/diffdrive/C4W.STL; visual mesh filename=package://mim_robots/meshes/diffdrive/C4W.STL
- link PW1: mass 0.0720898510112747 -> 0.0290199529351017; geometry collision mesh filename=package://mim_robots/meshes/diffdrive/PW1.STL; visual mesh filename=package://mim_robots/meshes/diffdrive/PW1.STL
- link PW2: mass 0.0720898510112747 -> 0.0290199529351017; geometry collision mesh filename=package://mim_robots/meshes/diffdrive/PW2.STL; visual mesh filename=package://mim_robots/meshes/diffdrive/PW2.STL
- link base_link: mass 2.38519315841668 -> 33.5973988123837; geometry collision mesh filename=package://mim_robots/meshes/diffdrive/base_link.STL; visual mesh filename=package://mim_robots/meshes/diffdrive/base_link.STL
Joints:
- removed joint C1J
- removed joint C1WJ
- removed joint C2J
- removed joint C2WJ
- removed joint C3J
- removed joint C3WJ
- removed joint C4J
- removed joint C4WJ
- removed joint PW1J
- removed joint PW2J
- added joint C1W_J: type continuous, parent C1, child C1W, origin xyz=-0.0210069660112502 -0.0865 0 rpy=-3.0886194316909 0 -1.5707963267949, axis 0 0.0529484501323336 0.998597246956241
- added joint C1_J: type continuous, parent base_link, child C1, origin xyz=0.337499999999999 -0.178513749758133 0.124000000000001 rpy=1.57079632679489 0 0.0264866109494407, axis 0 1 0
- added joint C2W_J: type continuous, parent C2, child C2W, origin xyz=-0.0210069660112502 -0.0865 0 rpy=-3.0886194316909 0 -1.5707963267949, axis 0 0.0529484501323336 0.998597246956241
- added joint C2_J: type continuous, parent base_link, child C2, origin xyz=0.337500000000001 0.176486250241866 0.123999999999999 rpy=1.57079632679489 0 0.0264866109494407, axis 0 1 0
- added joint C3W_J: type continuous, parent C3, child C3W, origin xyz=-0.02100696601125 -0.0865 0 rpy=-3.0886194316909 0 -1.5707963267949, axis 0 0.0529484501323336 0.998597246956241
- added joint C3_J: type continuous, parent base_link, child C3, origin xyz=-0.337499999999999 0.176486250241869 0.123999999999999 rpy=1.57079632679489 0 0.0264866109494407, axis 0 1 0
- added joint C4W_J: type continuous, parent C4, child C4W, origin xyz=-0.02100696601125 -0.0864999999999998 0 rpy=-3.0886194316909 0 -1.5707963267949, axis 0 0.0529484501323336 0.998597246956241
- added joint C4_J: type continuous, parent base_link, child C4, origin xyz=-0.337500000000001 -0.178513749758131 0.123997864045001 rpy=1.57079632679489 0 0.0264866109494407, axis 0 1 0
- added joint LIDAR_J: type fixed, parent base_link, child LIDAR, origin xyz=0.321103295710635 -0.000963772085925339 0.384500000000008 rpy=1.57079632679489 0 -3.14159265358979, axis 0 0 0
- added joint PW1_J: type continuous, parent base_link, child PW1, origin xyz=0 -0.200513749758132 0.0375000000000016 rpy=1.57079632679489 1.5707963267949 0, axis 0 0 1
- added joint PW2_J: type continuous, parent base_link, child PW2, origin xyz=0 0.198486250241876 0.0374999999999999 rpy=1.57079632679489 1.5707963267949 0, axis 0 0 1

File: urdf/diffdrive_arm.xacro (robot description, xacro)
@@ -14,31 +14,18 @@
       xyz="0 0 0" />
   </joint>
-  <!-- <xacro:include filename="$(find mim_robots)/urdf/mim_arm.urdf"/> -->
-  <!--  -->
-  <!-- <joint name="car_to_arm" type="fixed"> -->
-  <!--   <origin -->
-  <!--     xyz="-0.2 0 0.281" -->
-  <!--     rpy="0 0 0" /> -->
-  <!--   <parent -->
-  <!--     link="base_link" /> -->
-  <!--   <child -->
-  <!--     link="mim_arm_base_link" /> -->
-  <!--   <axis -->
-  <!--     xyz="0 0 0" /> -->
-  <!-- </joint> -->
-  <!-- <link name="world"></link> -->
-  <!-- <joint name="world_to_arm" type="fixed"> -->
-  <!--   <origin -->
-  <!--     xyz="0 0 0" -->
-  <!--     rpy="0 0 0" /> -->
-  <!--   <parent -->
-  <!--     link="world" /> -->
-  <!--   <child -->
-  <!--     link="mim_arm_base_link" /> -->
-  <!--   <axis -->
-  <!--     xyz="0 0 0" /> -->
-  <!-- </joint> -->
+  <xacro:include filename="$(find mim_robots)/urdf/arm/mim_arm.urdf"/>
+  <joint name="car_to_arm" type="fixed">
+    <origin
+      xyz="-0.2 0 0.281"
+      rpy="0 0 0" />
+    <parent
+      link="base_link" />
+    <child
+      link="arm_base_link" />
+    <axis
+      xyz="0 0 0" />
+  </joint>
   <xacro:include filename="$(find mim_robots)/urdf/gazebo/diffdrive_arm.gazebo"/>
   <xacro:include filename="$(find mim_robots)/urdf/diffdrive/diffdrive_transmission.urdf"/>
-  <!-- <xacro:include filename="$(find mim_robots)/urdf/arm_transmission.urdf"/> -->
+  <xacro:include filename="$(find mim_robots)/urdf/arm/arm_transmission.urdf"/>
 </robot>

File: urdf/rockerb/mim_rockerb.urdf (robot description, URDF)
Before this commit: robot mim_rockerb, 13 links, 12 joints
Links:
- added link LIDAR, mass 0.0730843681136202; collision mesh filename=package://mim_robots/meshes/rockerb/LIDAR.STL; visual mesh filename=package://mim_robots/meshes/rockerb/LIDAR.STL
- link B1: mass 0.53077264293737 -> 4.13605312852322; geometry collision mesh filename=package://mim_robots/meshes/rockerb/B1.STL; visual mesh filename=package://mim_robots/meshes/rockerb/B1.STL
- link B2: mass 0.53077264293737 -> 4.13605312852322; geometry collision mesh filename=package://mim_robots/meshes/rockerb/B2.STL; visual mesh filename=package://mim_robots/meshes/rockerb/B2.STL
- link C1: mass 0.0175932153888398 -> 0.13722708003295; geometry collision mesh filename=package://mim_robots/meshes/rockerb/C1.STL; visual mesh filename=package://mim_robots/meshes/rockerb/C1.STL
- link C2: mass 0.0175932153888397 -> 0.137227080032951; geometry collision mesh filename=package://mim_robots/meshes/rockerb/C2.STL; visual mesh filename=package://mim_robots/meshes/rockerb/C2.STL
- link C3: mass 0.0175932153888398 -> 0.13722708003295; geometry collision mesh filename=package://mim_robots/meshes/rockerb/C3.STL; visual mesh filename=package://mim_robots/meshes/rockerb/C3.STL
- link C4: mass 0.0175932153888396 -> 0.13722708003295; geometry collision mesh filename=package://mim_robots/meshes/rockerb/C4.STL; visual mesh filename=package://mim_robots/meshes/rockerb/C4.STL
- link CW1: geometry collision mesh filename=package://mim_robots/meshes/rockerb/CW1.STL; visual mesh filename=package://mim_robots/meshes/rockerb/CW1.STL
- link CW2: geometry collision mesh filename=package://mim_robots/meshes/rockerb/CW2.STL; visual mesh filename=package://mim_robots/meshes/rockerb/CW2.STL
- link CW3: geometry collision mesh filename=package://mim_robots/meshes/rockerb/CW3.STL; visual mesh filename=package://mim_robots/meshes/rockerb/CW3.STL
- link CW4: geometry collision mesh filename=package://mim_robots/meshes/rockerb/CW4.STL; visual mesh filename=package://mim_robots/meshes/rockerb/CW4.STL
- link P1: geometry collision mesh filename=package://mim_robots/meshes/rockerb/P1.STL; visual mesh filename=package://mim_robots/meshes/rockerb/P1.STL
- link P2: geometry collision mesh filename=package://mim_robots/meshes/rockerb/P2.STL; visual mesh filename=package://mim_robots/meshes/rockerb/P2.STL
- link base_link: mass 0.858306725756551 -> 24.5477793824158; geometry collision mesh filename=package://mim_robots/meshes/rockerb/base_link.STL; visual mesh filename=package://mim_robots/meshes/rockerb/base_link.STL
Joints:
- removed joint b1_j
- removed joint b2_j
- removed joint c1_j
- removed joint c2_j
- removed joint c3_j
- removed joint c4_j
- removed joint cw1_j
- removed joint cw2_j
- removed joint cw3_j
- removed joint cw4_j
- removed joint p1_j
- removed joint p2_j
- added joint B1_J: type continuous, parent base_link, child B1, origin xyz=0.158749999999996 -0.0785137497581288 0.144999999999991 rpy=1.57079632679489 0 -3.14159265358979, axis 0 0 1
- added joint B2_J: type continuous, parent base_link, child B2, origin xyz=0.158749999999999 0.0764862502418753 0.144999999999991 rpy=1.5707963267949 0 3.14159265358979, axis 0 0 1
- added joint C1_J: type continuous, parent B1, child C1, origin xyz=-0.178749999999958 -0.0210000000003531 -0.100000000000004 rpy=-3.14159265358973 -0.026486610949433 3.14159265358979, axis 0 1 0
- added joint C2_J: type continuous, parent B2, child C2, origin xyz=-0.178749999999998 -0.0209999999999919 0.0999999999999913 rpy=-3.14159265358979 -0.02648661094944 3.14159265358979, axis 0 1 0
- added joint C3_J: type continuous, parent base_link, child C3, origin xyz=-0.3375 0.17648625024187 0.123999999999991 rpy=1.5707963267949 0 0.0264866109494337, axis 0 1 0
- added joint C4_J: type continuous, parent base_link, child C4, origin xyz=-0.337500000000004 -0.17851374975813 0.12399786404499 rpy=1.5707963267949 0 0.0264866109494337, axis 0 1 0
- added joint CW1_J: type continuous, parent C1, child CW1, origin xyz=-0.0210069660114238 -0.0864999999999466 0 rpy=-3.0886194316909 0 -1.5707963267949, axis 0 0.0529484501323336 0.998597246956241
- added joint CW2_J: type continuous, parent C2, child CW2, origin xyz=-0.0210069660112452 -0.0864999999999993 0 rpy=-3.0886194316909 0 -1.5707963267949, axis 0 0.0529484501323336 0.998597246956241
- added joint CW3_J: type continuous, parent C3, child CW3, origin xyz=-0.02100696601125 -0.0865 0 rpy=-3.0886194316909 0 -1.5707963267949, axis 0 0.0529484501323336 0.998597246956241
- added joint CW4_J: type continuous, parent C4, child CW4, origin xyz=-0.0210069660112505 -0.0864999999999983 0 rpy=-3.0886194316909 0 -1.5707963267949, axis 0 0.0529484501323336 0.998597246956241
- added joint LIDAR_J: type fixed, parent base_link, child LIDAR, origin xyz=0.317603295710605 -0.000963772085933554 0.338499999999593 rpy=1.5707963267949 0 3.14159265358979, axis 0 0 0
- added joint P1_J: type continuous, parent B1, child P1, origin xyz=0.15875 -0.107499999999674 -0.122 rpy=0 0 -1.5707963267949, axis 0 0 1
- added joint P2_J: type continuous, parent B2, child P2, origin xyz=0.15875 -0.107499999999987 0.122000000000001 rpy=0 0 -1.5707963267949, axis 0 0 1

File: urdf/rockerb_arm.xacro (robot description, xacro)
@@ -14,30 +14,18 @@
       xyz="0 0 0" />
   </joint>
-  <!-- <xacro:include filename="$(find mim_robots)/urdf/mim_arm.urdf"/> -->
-  <!-- <joint name="car_to_arm" type="fixed"> -->
-  <!--   <origin -->
-  <!--     xyz="-0.2 0 0.281" -->
-  <!--     rpy="0 0 0" /> -->
-  <!--   <parent -->
-  <!--     link="base_link" /> -->
-  <!--   <child -->
-  <!--     link="mim_arm_base_link" /> -->
-  <!--   <axis -->
-  <!--     xyz="0 0 0" /> -->
-  <!-- </joint> -->
-  <!-- <link name="world"></link> -->
-  <!-- <joint name="world_to_arm" type="fixed"> -->
-  <!--   <origin -->
-  <!--     xyz="0 0 0" -->
-  <!--     rpy="0 0 0" /> -->
-  <!--   <parent -->
-  <!--     link="world" /> -->
-  <!--   <child -->
-  <!--     link="mim_arm_base_link" /> -->
-  <!--   <axis -->
-  <!--     xyz="0 0 0" /> -->
-  <!-- </joint> -->
+  <xacro:include filename="$(find mim_robots)/urdf/arm/mim_arm.urdf"/>
+  <joint name="car_to_arm" type="fixed">
+    <origin
+      xyz="-0.2 0 0.281"
+      rpy="0 0 0" />
+    <parent
+      link="base_link" />
+    <child
+      link="arm_base_link" />
+    <axis
+      xyz="0 0 0" />
+  </joint>
   <xacro:include filename="$(find mim_robots)/urdf/gazebo/rockerb_arm.gazebo"/>
   <xacro:include filename="$(find mim_robots)/urdf/rockerb/rockerb_transmission.urdf"/>
-  <!-- <xacro:include filename="$(find mim_robots)/urdf/arm_transmission.urdf"/> -->
+  <xacro:include filename="$(find mim_robots)/urdf/arm/arm_transmission.urdf"/>
 </robot>
