Commit message: Remove unused code

File: urdf/diffdrive_arm.xacro (robot description, xacro)
@@ -2,5 +2,6 @@
 <robot name="mim_diffdrive_arm" xmlns:xacro="http://www.ros.org/wiki/xacro">
   <xacro:include filename="$(find mim_robots)/urdf/diffdrive/mim_diffdrive.urdf"/>
-  <link name="world"></link>
+  <xacro:arg name="dummy_link" default="dummy_link"/>
+  <link name="$(arg dummy_link)"></link>
   <joint name="dummy_to_car" type="fixed">
     <origin
@@ -8,5 +9,5 @@
       rpy="0 0 0" />
     <parent
-      link="world" />
+      link="$(arg dummy_link)" />
     <child
       link="base_link" />
