Commit message: Fix ramp urdf relative path

File: urdf/other_models/ramp.urdf (robot description, URDF)
Before this commit: robot ramp, 2 links, 1 joints
Links:
- link base_link: geometry collision mesh filename=package://mim_robots/meshes/ramp/base_link.STL; visual mesh filename=package://mim_robots/meshes/ramp/base_link.STL
