Commit message: Add arm pick script

File: urdf/arm/mim_arm.urdf (robot description, URDF)
Before this commit: robot mim_arm, 9 links, 8 joints
Joints:
- joint J1: limit lower=-2 upper=2 effort=500 velocity=30 -> lower=-2 upper=2 effort=500 velocity=15
- joint J2: limit lower=-2 upper=2 effort=500 velocity=30 -> lower=-2 upper=2 effort=500 velocity=15
- joint J3: limit lower=-2 upper=2 effort=1000 velocity=30 -> lower=-2 upper=2 effort=1000 velocity=15
- joint J4: limit lower=-2 upper=2 effort=500 velocity=30 -> lower=-2 upper=2 effort=500 velocity=15
- joint J5: limit lower=-2 upper=2 effort=1000 velocity=30 -> lower=-2 upper=2 effort=1000 velocity=15

File: urdf/diffdrive_arm.xacro (robot description, xacro)
@@ -2,5 +2,5 @@
 <robot name="mim_diffdrive_arm" xmlns:xacro="http://www.ros.org/wiki/xacro">
   <xacro:include filename="$(find mim_robots)/urdf/diffdrive/mim_diffdrive.urdf"/>
-  <link name="dummy_link"></link>
+  <link name="world"></link>
   <joint name="dummy_to_car" type="fixed">
     <origin
@@ -8,5 +8,5 @@
       rpy="0 0 0" />
     <parent
-      link="dummy_link" />
+      link="world" />
     <child
       link="base_link" />

Commit message: Finish pick and place script
Add script function for calculating the inverse velocity
The pick and place start from moving to a pick pose then
go straight downward to grasp the objects then reverse

Fix the diffdrive empty wheels

File: urdf/arm/mim_arm.urdf (robot description, URDF)
Before this commit: robot mim_arm, 9 links, 8 joints
Joints:
- joint J1: limit lower=-2 upper=2 effort=500 velocity=15 -> lower=-2 upper=2 effort=500 velocity=1
- joint J2: limit lower=-2 upper=2 effort=500 velocity=15 -> lower=-2 upper=2 effort=500 velocity=1
- joint J3: limit lower=-2 upper=2 effort=1000 velocity=15 -> lower=-2 upper=2 effort=1000 velocity=1
- joint J4: limit lower=-2 upper=2 effort=500 velocity=15 -> lower=-2 upper=2 effort=500 velocity=1
- joint J5: limit lower=-2 upper=2 effort=1000 velocity=15 -> lower=-2 upper=2 effort=1000 velocity=1
- joint J6: axis 0 0 0 -> 1 0 0; limit (none) -> lower=-2 upper=2 effort=1000 velocity=1; type fixed -> continuous

File: urdf/diffdrive/mim_diffdrive.urdf (robot description, URDF)
Before this commit: robot mim_diffdrive, 12 links, 11 joints
Links:
- removed link PW1
- removed link PW2
- added link P1, mass 0.0720898510112747; collision mesh filename=package://mim_robots/meshes/diffdrive/P1.STL; visual mesh filename=package://mim_robots/meshes/diffdrive/P1.STL
- added link P2, mass 0.0720898510112747; collision mesh filename=package://mim_robots/meshes/diffdrive/P2.STL; visual mesh filename=package://mim_robots/meshes/diffdrive/P2.STL
- link C1: mass 0.133845469700625 -> 0.13722708003295
- link C1W: mass 0.0290199529351017 -> 0.0741004703095722
- link C2: mass 0.133845469700627 -> 0.137227080032951
- link C2W: mass 0.0290199529351017 -> 0.0741004703095722
- link C3: mass 0.133845469700626 -> 0.137227080032949
- link C3W: mass 0.0290199529351017 -> 0.0741004703095722
- link C4: mass 0.133845469700625 -> 0.13722708003295
- link C4W: mass 0.0290199529351017 -> 0.0741004703095722
- link LIDAR: mass 0.0730843683225071 -> 0.0730843682728084
Joints:
- removed joint PW1_J
- removed joint PW2_J
- added joint P1_J: type continuous, parent base_link, child P1, origin xyz=0 -0.210513749758133 0.0375000000000007 rpy=1.57079632679489 1.5707963267949 0, axis 0 0 1
- added joint P2_J: type continuous, parent base_link, child P2, origin xyz=0 0.208486250241876 0.0375000000000008 rpy=1.57079632679489 1.5707963267949 0, axis 0 0 1
- joint C1W_J: origin xyz=-0.0210069660112502 -0.0865 0 rpy=-3.0886194316909 0 -1.5707963267949 -> xyz=-0.0210069660112502 0.00702786404500044 0 rpy=-3.0886194316909 0 -1.5707963267949
- joint C1_J: origin xyz=0.337499999999999 -0.178513749758133 0.124000000000001 rpy=1.57079632679489 0 0.0264866109494407 -> xyz=0.337499999999999 -0.178513749758134 0.0304721359549996 rpy=1.5707963267949 0 0.0264866109494407
- joint C2W_J: origin xyz=-0.0210069660112502 -0.0865 0 rpy=-3.0886194316909 0 -1.5707963267949 -> xyz=-0.0210069660112502 0.00702786404500046 0 rpy=-3.0886194316909 0 -1.5707963267949
- joint C2_J: origin xyz=0.337500000000001 0.176486250241866 0.123999999999999 rpy=1.57079632679489 0 0.0264866109494407 -> xyz=0.337500000000001 0.176486250241866 0.0304721359549995 rpy=1.5707963267949 0 0.0264866109494407
- joint C3W_J: origin xyz=-0.02100696601125 -0.0865 0 rpy=-3.0886194316909 0 -1.5707963267949 -> xyz=-0.02100696601125 0.00702786404500066 0 rpy=-3.0886194316909 0 -1.5707963267949
- joint C3_J: origin xyz=-0.337499999999999 0.176486250241869 0.123999999999999 rpy=1.57079632679489 0 0.0264866109494407 -> xyz=-0.337500000000001 -0.178513749758132 0.0304699999999996 rpy=1.5707963267949 0 0.0264866109494407
- joint C4W_J: origin xyz=-0.02100696601125 -0.0864999999999998 0 rpy=-3.0886194316909 0 -1.5707963267949 -> xyz=-0.02100696601125 0.00702786404500043 0 rpy=-3.0886194316909 0 -1.5707963267949
- joint C4_J: origin xyz=-0.337500000000001 -0.178513749758131 0.123997864045001 rpy=1.57079632679489 0 0.0264866109494407 -> xyz=-0.337499999999999 0.176486250241868 0.0304721359549995 rpy=1.5707963267949 0 0.0264866109494407
- joint LIDAR_J: origin xyz=0.321103295710635 -0.000963772085925339 0.384500000000008 rpy=1.57079632679489 0 -3.14159265358979 -> xyz=0.321103295710635 -0.000963772085875598 0.374500000000008 rpy=1.57079632679489 0 -3.14159265358979

File: urdf/diffdrive_arm.xacro (robot description, xacro)
@@ -18,5 +18,5 @@
   <joint name="car_to_arm" type="fixed">
     <origin
-      xyz="-0.2 0 0.281"
+      xyz="-0.2 0 0.321"
       rpy="0 0 0" />
     <parent

File: urdf/rockerb_arm.xacro (robot description, xacro)
@@ -17,5 +17,5 @@
   <joint name="car_to_arm" type="fixed">
     <origin
-      xyz="-0.2 0 0.281"
+      xyz="-0.2 0 0.285"
       rpy="0 0 0" />
     <parent
